File: usb_amp/usb_amp.sch (KiCad schematic (older format))
At the start: 0 parts

Commit message: Continue routing top level diagram
Other:
- note added: "10k in, low-z out"
- note added: "12->19 V, \n60->100 W"
- note added: "CS3318?"
- note added: "DGND and AGND\nreferenced here"
- note added: "ISL54405"
- note added: "Powered by USB"
- note added: "Signals referenced\nto AGND here"
